Commit message: s2s well

File: description/robots/ehr03/urdf/ehr03.urdf (robot description, URDF)
Before this commit: robot ehr_03, 32 links, 31 joints
Joints:
- joint l_arm_1: limit lower=-3.58 upper=2.71 effort=60 velocity=15.603 -> lower=-3.58 upper=2.71 effort=30 velocity=15.603
- joint l_arm_2: limit lower=-0.174 upper=2.966 effort=75 velocity=12.252 -> lower=-0.174 upper=2.966 effort=40 velocity=12.252
- joint l_arm_3: limit lower=-1.57 upper=1.57 effort=36 velocity=3 -> lower=-1.57 upper=1.57 effort=20 velocity=3
- joint l_arm_4: limit lower=-1.74 upper=0.785 effort=36 velocity=9.320 -> lower=-1.74 upper=0.785 effort=20 velocity=9.320
- joint l_arm_5: limit lower=-0.37 upper=0.37 effort=36 velocity=9.320 -> lower=-0.37 upper=0.37 effort=20 velocity=9.320
- joint l_arm_6: limit lower=-0.37 upper=0.385 effort=36 velocity=3 -> lower=-0.37 upper=0.385 effort=20 velocity=3
- joint l_leg_1: limit lower=-1.57 upper=1.57 effort=320 velocity=14.137 -> lower=-1.57 upper=1.57 effort=160 velocity=14.137
- joint l_leg_2: limit lower=-0.2 upper=1.57 effort=150 velocity=14.661 -> lower=-0.2 upper=1.57 effort=100 velocity=14.661
- joint l_leg_3: limit lower=-1.57 upper=1.57 effort=150 velocity=14.661 -> lower=-1.57 upper=1.57 effort=100 velocity=14.661
- joint l_leg_4: limit lower=-0.523 upper=1.57 effort=320 velocity=14.137 -> lower=-0.523 upper=1.57 effort=160 velocity=14.137
- joint l_leg_5: limit lower=-0.84 upper=0.7 effort=75 velocity=12.252 -> lower=-0.84 upper=0.7 effort=40 velocity=12.252
- joint l_leg_6: limit lower=-0.45 upper=0.45 effort=75 velocity=12.252 -> lower=-0.45 upper=0.45 effort=40 velocity=12.252
- joint r_arm_1: limit lower=-3.58 upper=2.71 effort=60 velocity=15.603 -> lower=-3.58 upper=2.71 effort=30 velocity=15.603
- joint r_arm_2: limit lower=-2.966 upper=0.174 effort=75 velocity=12.252 -> lower=-2.966 upper=0.174 effort=40 velocity=12.252
- joint r_arm_3: limit lower=-1.57 upper=1.57 effort=36 velocity=3 -> lower=-1.57 upper=1.57 effort=20 velocity=3
- joint r_arm_4: limit lower=-1.74 upper=0.785 effort=36 velocity=9.320 -> lower=-1.74 upper=0.785 effort=20 velocity=9.320
- joint r_arm_5: limit lower=-0.37 upper=0.37 effort=36 velocity=9.320 -> lower=-0.37 upper=0.37 effort=20 velocity=9.320
- joint r_arm_6: limit lower=-0.385 upper=0.37 effort=36 velocity=3 -> lower=-0.385 upper=0.37 effort=20 velocity=3
- joint r_leg_1: limit lower=-1.57 upper=1.57 effort=320 velocity=14.137 -> lower=-1.57 upper=1.57 effort=160 velocity=14.137
- joint r_leg_2: limit lower=-1.57 upper=0.2 effort=150 velocity=14.661 -> lower=-1.57 upper=0.2 effort=100 velocity=14.661
- joint r_leg_3: limit lower=-1.57 upper=1.57 effort=150 velocity=14.661 -> lower=-1.57 upper=1.57 effort=100 velocity=14.661
- joint r_leg_4: limit lower=-0.523 upper=1.57 effort=320 velocity=14.137 -> lower=-0.523 upper=1.57 effort=160 velocity=14.137
- joint r_leg_5: limit lower=-0.84 upper=0.7 effort=75 velocity=12.252 -> lower=-0.84 upper=0.7 effort=40 velocity=12.252
- joint r_leg_6: limit lower=-0.45 upper=0.45 effort=75 velocity=12.252 -> lower=-0.45 upper=0.45 effort=40 velocity=12.252
